Commit message: [fix] change tf_frame config

File: turtlebot3/urdf/turtlebot3_waffle_mid360.gazebo.xacro (robot description, xacro)
@@ -148,5 +148,5 @@
     <gazebo reference="livox_scan">
       <material>Gazebo/FlatBlack</material>
-      <sensor type="ray" name="livox_mid360">
+      <sensor type="ray" name="livox_scan">
         <pose>0 0 0 0 0 0</pose>
         <visualize>True</visualize>

File: turtlebot3/urdf/turtlebot3_waffle_mid360.urdf.xacro (robot description, xacro)
@@ -191,6 +191,6 @@
       <parent link="base_link"/>
       <child link="livox_scan"/>
-      <origin rpy="0 0 1.5707"
-              xyz="-0.05 0.0 0.12"/>
+      <origin rpy="0 0 0"
+              xyz="-0.05 0.0 0.09"/>
   </joint>
 </robot>
